Commit message: スクリプト整理

File: ros2_ws/src/ai_ship_robot_description/urdf/ai_ship_robot.urdf.xacro (robot description, xacro)
@@ -112,6 +112,8 @@
        lidar_pattern_single.urdf.urdf.xacro
        ================================================================ -->
-  <!-- <xacro:include filename="lidar_pattern_dual.urdf.xacro" /> -->
-  <xacro:include filename="lidar_pattern_single.urdf.xacro" />
+  <!-- <xacro:include filename="lidar_pattern_dual_out20.urdf.xacro" /> -->
+  <!-- <xacro:include filename="lidar_pattern_dual_out38.urdf.xacro" /> -->
+  <xacro:include filename="lidar_pattern_dual_updown.urdf.xacro" />
+  <!-- <xacro:include filename="lidar_pattern_single.urdf.xacro" /> -->
   <link name="imu_link">
     <visual>
@@ -141,25 +143,27 @@
   </gazebo>
   <xacro:if value="$(arg use_sim)">
+    <!-- Gazebo Classic上で平面移動とodom/TFを再現する。 -->
     <gazebo>
-      <plugin name="planar_move_controller" filename="libgazebo_ros_planar_move.so">
+      <plugin filename="libgazebo_ros_planar_move.so" name="gazebo_ros_planar_move">
         <ros>
-          <remapping>cmd_vel:=cmd_vel</remapping>
-          <remapping>odom:=odom</remapping>
+          <namespace>/</namespace>
         </ros>
-        <update_rate>100.0</update_rate>
-        <publish_rate>30.0</publish_rate>
+        <command_topic>cmd_vel</command_topic>
+        <odometry_topic>odom</odometry_topic>
+        <odometry_frame>odom</odometry_frame>
+        <robot_base_frame>base_footprint</robot_base_frame>
         <publish_odom>true</publish_odom>
         <publish_odom_tf>true</publish_odom_tf>
-        <odometry_frame>odom</odometry_frame>
-        <robot_base_frame>base_footprint</robot_base_frame>
       </plugin>
     </gazebo>
+    <!-- IMUはClassicのgazebo_ros sensor plugin経由でROS topicへ流す。 -->
     <gazebo reference="imu_link">
       <sensor name="imu" type="imu">
         <always_on>true</always_on>
         <update_rate>100</update_rate>
-        <plugin name="imu_controller" filename="libgazebo_ros_imu_sensor.so">
+        <plugin filename="libgazebo_ros_imu_sensor.so" name="gazebo_ros_imu_sensor">
           <ros>
-            <remapping>~/out:=/imu/data</remapping>
+            <namespace>/</namespace>
+            <remapping>~/out:=imu/data</remapping>
           </ros>
           <frame_name>imu_link</frame_name>

File: ros2_ws/src/ai_ship_robot_description/urdf/mid360_lidar.urdf.xacro (robot description, xacro)
@@ -2,59 +2,64 @@
 <robot xmlns:xacro="http://www.ros.org/wiki/xacro" name="mid360_lidar">
   <xacro:arg name="half_lidar_resolution" default="false" />
+  <xacro:arg name="quarter_lidar_resolution" default="false" />
   <xacro:property name="mid360_depth" value="0.060" />
   <xacro:property name="mid360_width" value="0.065" />
   <xacro:property name="mid360_height" value="0.065" />
-  <xacro:property name="mid360_horizontal_samples" value="500" />
-  <xacro:property name="mid360_vertical_samples" value="40" />
-  <xacro:property name="mid360_half_horizontal_samples" value="250" />
-  <xacro:property name="mid360_half_vertical_samples" value="20" />
+  <xacro:property name="mid360_samples" value="40000" />
+  <xacro:property name="mid360_downsample" value="1" />
+  <xacro:property name="mid360_half_downsample" value="2" />
+  <xacro:property name="mid360_quarter_downsample" value="4" />
   <xacro:macro name="mid360_gazebo_sensor" params="prefix">
     <gazebo reference="${prefix}_lidar_link">
-      <sensor name="${prefix}_livox_mid360" type="ray">
+      <sensor name="${prefix}_lidar_link" type="ray">
         <always_on>true</always_on>
         <visualize>false</visualize>
         <update_rate>10</update_rate>
-        <ray>
-          <scan>
-            <horizontal>
-              <xacro:unless value="$(arg half_lidar_resolution)">
-                <samples>${mid360_horizontal_samples}</samples>
-              </xacro:unless>
-              <xacro:if value="$(arg half_lidar_resolution)">
-                <samples>${mid360_half_horizontal_samples}</samples>
-              </xacro:if>
-              <resolution>1</resolution>
-              <min_angle>-${pi}</min_angle>
-              <max_angle>${pi}</max_angle>
-            </horizontal>
-            <vertical>
-              <xacro:unless value="$(arg half_lidar_resolution)">
-                <samples>${mid360_vertical_samples}</samples>
-              </xacro:unless>
-              <xacro:if value="$(arg half_lidar_resolution)">
-                <samples>${mid360_half_vertical_samples}</samples>
-              </xacro:if>
-              <resolution>1</resolution>
-              <min_angle>${-7.0 * pi / 180.0}</min_angle>
-              <max_angle>${52.0 * pi / 180.0}</max_angle>
-            </vertical>
-          </scan>
-          <range>
-            <min>0.10</min>
-            <max>40.0</max>
-            <resolution>0.02</resolution>
-          </range>
-          <noise>
-            <type>gaussian</type>
-            <mean>0.0</mean>
-            <stddev>0.0</stddev>
-          </noise>
-        </ray>
-        <plugin name="${prefix}_lidar_3d_controller" filename="libgazebo_ros_ray_sensor.so">
-          <ros>
-            <remapping>~/out:=/${prefix}_lidar/points</remapping>
-          </ros>
-          <output_type>sensor_msgs/PointCloud2</output_type>
-          <frame_name>${prefix}_lidar_link</frame_name>
+        <!-- Livox pluginの要求に合わせ、可視化用のray設定とCSV走査設定を同居させる。 -->
+        <plugin name="${prefix}_livox_plugin" filename="libros2_livox.so">
+          <ray>
+            <scan>
+              <horizontal>
+                <samples>100</samples>
+                <resolution>1</resolution>
+                <min_angle>0</min_angle>
+                <max_angle>${2.0 * pi}</max_angle>
+              </horizontal>
+              <vertical>
+                <samples>360</samples>
+                <resolution>1</resolution>
+                <min_angle>${-7.22 * pi / 180.0}</min_angle>
+                <max_angle>${55.22 * pi / 180.0}</max_angle>
+              </vertical>
+            </scan>
+            <range>
+              <min>0.10</min>
+              <max>200.0</max>
+              <resolution>0.002</resolution>
+            </range>
+            <noise>
+              <type>gaussian</type>
+              <mean>0.0</mean>
+              <stddev>0.01</stddev>
+            </noise>
+          </ray>
+          <visualize>false</visualize>
+          <samples>${mid360_samples}</samples>
+          <!-- downsample値だけでLivox pluginの負荷を切り替え、topic構成は維持する。 -->
+          <xacro:if value="$(arg quarter_lidar_resolution)">
+            <downsample>${mid360_quarter_downsample}</downsample>
+          </xacro:if>
+          <xacro:unless value="$(arg half_lidar_resolution)">
+            <xacro:unless value="$(arg quarter_lidar_resolution)">
+              <downsample>${mid360_downsample}</downsample>
+            </xacro:unless>
+          </xacro:unless>
+          <xacro:if value="$(arg half_lidar_resolution)">
+            <downsample>${mid360_half_downsample}</downsample>
+          </xacro:if>
+          <csv_file_name>$(find ros2_livox_simulation)/scan_mode/mid360.csv</csv_file_name>
+          <topic>${prefix}_livox</topic>
+          <custom_topic>/${prefix}_lidar/custom</custom_topic>
+          <pointcloud2_topic>/${prefix}_lidar/points</pointcloud2_topic>
         </plugin>
       </sensor>

Commit message: 高速化と整理

File: ros2_ws/src/ai_ship_robot_description/urdf/ai_ship_robot.urdf.xacro (robot description, xacro)
@@ -11,4 +11,13 @@
   <xacro:property name="wheel_x_offset" value="${base_length / 2.0 - wheel_radius - 0.02}" />
   <xacro:property name="base_center_z" value="${ground_clearance - wheel_radius + base_height / 2.0}" />
+  <xacro:property name="arm_robot_body_length" value="0.62" />
+  <xacro:property name="arm_robot_body_width" value="0.62" />
+  <xacro:property name="arm_robot_body_height" value="0.74" />
+  <xacro:property name="arm_robot_arm_radius" value="0.05" />
+  <xacro:property name="arm_robot_upper_arm_length" value="0.60" />
+  <xacro:property name="arm_robot_forearm_length" value="0.50" />
+  <xacro:property name="arm_robot_wrist_length" value="0.40" />
+  <xacro:property name="arm_robot_first_arm_pitch" value="${45.0 * pi / 180.0}" />
+  <xacro:property name="arm_robot_second_arm_pitch" value="${115.0 * pi / 180.0}" />
   <xacro:macro name="box_inertia" params="mass x y z">
     <inertial>
@@ -79,4 +88,101 @@
     </gazebo>
   </xacro:macro>
+  <xacro:macro name="fixed_arm_robot_fixture">
+    <!-- LiDAR遮蔽を見やすくするため、上物本体は台車より一回り小さい箱で高さを強調する。 -->
+    <link name="arm_robot_body_link">
+      <visual>
+        <origin xyz="0 0 0" rpy="0 0 0" />
+        <geometry>
+          <box size="${arm_robot_body_length} ${arm_robot_body_width} ${arm_robot_body_height}" />
+        </geometry>
+        <material name="arm_robot_green">
+          <color rgba="0.10 0.45 0.16 1.0" />
+        </material>
+      </visual>
+      <collision>
+        <origin xyz="0 0 0" rpy="0 0 0" />
+        <geometry>
+          <box size="${arm_robot_body_length} ${arm_robot_body_width} ${arm_robot_body_height}" />
+        </geometry>
+      </collision>
+      <xacro:box_inertia mass="18.0" x="${arm_robot_body_length}" y="${arm_robot_body_width}" z="${arm_robot_body_height}" />
+    </link>
+    <joint name="arm_robot_body_joint" type="fixed">
+      <parent link="base_link" />
+      <child link="arm_robot_body_link" />
+      <origin xyz="0 0 ${base_center_z + base_height / 2.0 + arm_robot_body_height / 2.0}" rpy="0 0 0" />
+    </joint>
+    <!-- 根元・肘・手首の3節を前方上がりに固定し、LiDARから見える外形を優先して再現する。 -->
+    <link name="arm_robot_upper_arm_link">
+      <visual>
+        <origin xyz="${arm_robot_upper_arm_length * cos(45.0 * pi / 180.0) / 2.0} 0 ${arm_robot_upper_arm_length * sin(45.0 * pi / 180.0) / 2.0}" rpy="0 ${arm_robot_first_arm_pitch} 0" />
+        <geometry>
+          <cylinder radius="${arm_robot_arm_radius}" length="${arm_robot_upper_arm_length}" />
+        </geometry>
+        <material name="arm_robot_blue">
+          <color rgba="0.12 0.42 0.62 1.0" />
+        </material>
+      </visual>
+      <collision>
+        <origin xyz="${arm_robot_upper_arm_length * cos(45.0 * pi / 180.0) / 2.0} 0 ${arm_robot_upper_arm_length * sin(45.0 * pi / 180.0) / 2.0}" rpy="0 ${arm_robot_first_arm_pitch} 0" />
+        <geometry>
+          <cylinder radius="${arm_robot_arm_radius}" length="${arm_robot_upper_arm_length}" />
+        </geometry>
+      </collision>
+      <xacro:cylinder_inertia mass="4.0" radius="${arm_robot_arm_radius}" length="${arm_robot_upper_arm_length}" axis="z" />
+    </link>
+    <joint name="arm_robot_shoulder_joint" type="fixed">
+      <parent link="arm_robot_body_link" />
+      <child link="arm_robot_upper_arm_link" />
+      <origin xyz="${arm_robot_body_length / 2.0} -0.10 ${0.20 - arm_robot_body_height / 2.0}" rpy="0 0 0" />
+    </joint>
+    <link name="arm_robot_forearm_link">
+      <visual>
+        <origin xyz="${arm_robot_forearm_length * cos(-25.0 * pi / 180.0) / 2.0} 0 ${arm_robot_forearm_length * sin(-25.0 * pi / 180.0) / 2.0}" rpy="0 ${arm_robot_second_arm_pitch} 0" />
+        <geometry>
+          <cylinder radius="${arm_robot_arm_radius}" length="${arm_robot_forearm_length}" />
+        </geometry>
+        <material name="arm_robot_blue">
+          <color rgba="0.12 0.42 0.62 1.0" />
+        </material>
+      </visual>
+      <collision>
+        <origin xyz="${arm_robot_forearm_length * cos(-25.0 * pi / 180.0) / 2.0} 0 ${arm_robot_forearm_length * sin(-25.0 * pi / 180.0) / 2.0}" rpy="0 ${arm_robot_second_arm_pitch} 0" />
+        <geometry>
+          <cylinder radius="${arm_robot_arm_radius}" length="${arm_robot_forearm_length}" />
+        </geometry>
+      </collision>
+      <xacro:cylinder_inertia mass="3.0" radius="${arm_robot_arm_radius}" length="${arm_robot_forearm_length}" axis="z" />
+    </link>
+    <!-- 関節位置を各アーム先端へ一致させ、指定された内角と鉛直手首を維持する。 -->
+    <joint name="arm_robot_elbow_joint" type="fixed">
+      <parent link="arm_robot_upper_arm_link" />
+      <child link="arm_robot_forearm_link" />
+      <origin xyz="${arm_robot_upper_arm_length * cos(45.0 * pi / 180.0)} 0 ${arm_robot_upper_arm_length * sin(45.0 * pi / 180.0)}" rpy="0 0 0" />
+    </joint>
+    <link name="arm_robot_wrist_link">
+      <visual>
+        <origin xyz="0 0 ${arm_robot_wrist_length / 2.0}" rpy="0 0 0" />
+        <geometry>
+          <cylinder radius="${arm_robot_arm_radius}" length="${arm_robot_wrist_length}" />
+        </geometry>
+        <material name="arm_robot_blue">
+          <color rgba="0.12 0.42 0.62 1.0" />
+        </material>
+      </visual>
+      <collision>
+        <origin xyz="0 0 ${arm_robot_wrist_length / 2.0}" rpy="0 0 0" />
+        <geometry>
+          <cylinder radius="${arm_robot_arm_radius}" length="${arm_robot_wrist_length}" />
+        </geometry>
+      </collision>
+      <xacro:cylinder_inertia mass="2.0" radius="${arm_robot_arm_radius}" length="${arm_robot_wrist_length}" axis="z" />
+    </link>
+    <joint name="arm_robot_wrist_joint" type="fixed">
+      <parent link="arm_robot_forearm_link" />
+      <child link="arm_robot_wrist_link" />
+      <origin xyz="${arm_robot_forearm_length * cos(-25.0 * pi / 180.0)} 0 ${arm_robot_forearm_length * sin(-25.0 * pi / 180.0)}" rpy="0 0 0" />
+    </joint>
+  </xacro:macro>
   <link name="base_footprint" />
   <joint name="base_footprint_joint" type="fixed">
@@ -107,4 +213,5 @@
   <xacro:drive_wheel prefix="right_front" x_position="${wheel_x_offset}" y_position="${-wheel_separation / 2.0}" />
   <xacro:drive_wheel prefix="right_rear" x_position="${-wheel_x_offset}" y_position="${-wheel_separation / 2.0}" />
+  <xacro:fixed_arm_robot_fixture />
   <!-- ==================== LiDAR installation pattern ====================
        Edit the filename below to switch LiDAR installation patterns.

Commit message: lidarのurdfをオプションで選択する

File: ros2_ws/src/ai_ship_robot_description/urdf/ai_ship_robot.urdf.xacro (robot description, xacro)
@@ -2,4 +2,5 @@
 <robot xmlns:xacro="http://www.ros.org/wiki/xacro" name="ai_ship_robot">
   <xacro:arg name="use_sim" default="true" />
+  <xacro:arg name="lidar_pattern_file" default="lidar_pattern_dual_updown.urdf.xacro" />
   <xacro:property name="base_length" value="0.72" />
   <xacro:property name="base_width" value="0.72" />
@@ -214,13 +215,6 @@
   <xacro:drive_wheel prefix="right_rear" x_position="${-wheel_x_offset}" y_position="${-wheel_separation / 2.0}" />
   <xacro:fixed_arm_robot_fixture />
-  <!-- ==================== LiDAR installation pattern ====================
-       Edit the filename below to switch LiDAR installation patterns.
-       lidar_pattern_dual.urdf.urdf.xacro
-       lidar_pattern_single.urdf.urdf.xacro
-       ================================================================ -->
-  <!-- <xacro:include filename="lidar_pattern_dual_out20.urdf.xacro" /> -->
-  <!-- <xacro:include filename="lidar_pattern_dual_out38.urdf.xacro" /> -->
-  <xacro:include filename="lidar_pattern_dual_updown.urdf.xacro" />
-  <!-- <xacro:include filename="lidar_pattern_single.urdf.xacro" /> -->
+  <!-- 起動時に指定された配置ファイルを読み込み、URDF編集なしでLiDARパターンを切り替える。 -->
+  <xacro:include filename="$(arg lidar_pattern_file)" />
   <link name="imu_link">
     <visual>

File: ros2_ws/src/ai_ship_robot_description/urdf/lidar_pattern_single.urdf.xacro (robot description, xacro)
@@ -8,5 +8,5 @@
   <xacro:property name="lidar_z" value="${base_center_z}" />
   <xacro:property name="lidar_roll" value="0.0" />
-  <xacro:property name="lidar_pitch" value="${30.0 * deg_to_rad}" />
+  <xacro:property name="lidar_pitch" value="${45.0 * deg_to_rad}" />
   <xacro:property name="lidar_yaw" value="0.0" />
   <xacro:mid360_lidar

Commit message: glim途中

File: ros2_ws/src/ai_ship_robot_description/urdf/ai_ship_robot.urdf.xacro (robot description, xacro)
@@ -3,4 +3,5 @@
   <xacro:arg name="use_sim" default="true" />
   <xacro:arg name="lidar_pattern_file" default="lidar_pattern_dual_updown.urdf.xacro" />
+  <xacro:arg name="publish_odom_tf" default="true" />
   <xacro:property name="base_length" value="0.72" />
   <xacro:property name="base_width" value="0.72" />
@@ -255,5 +256,5 @@
         <robot_base_frame>base_footprint</robot_base_frame>
         <publish_odom>true</publish_odom>
-        <publish_odom_tf>true</publish_odom_tf>
+        <publish_odom_tf>$(arg publish_odom_tf)</publish_odom_tf>
       </plugin>
     </gazebo>

File: ros2_ws/src/ai_ship_robot_description/urdf/lidar/models/mid360_lidar.urdf.xacro (robot description, xacro)
@@ -10,4 +10,8 @@
   <xacro:property name="mid360_half_downsample" value="2" />
   <xacro:property name="mid360_quarter_downsample" value="4" />
+  <xacro:property name="mid360_imu_x" value="0.011" />
+  <xacro:property name="mid360_imu_y" value="0.02329" />
+  <xacro:property name="mid360_imu_z" value="-0.04412" />
+  <xacro:property name="mid360_imu_size" value="0.015" />
   <xacro:macro name="mid360_gazebo_sensor" params="prefix">
     <gazebo reference="${prefix}_lidar_link">
@@ -66,5 +70,21 @@
     </gazebo>
   </xacro:macro>
-  <xacro:macro name="mid360_lidar" params="prefix x y z roll pitch yaw">
+  <xacro:macro name="mid360_gazebo_imu" params="prefix imu_topic">
+    <gazebo reference="${prefix}_lidar_imu_link">
+      <sensor name="${prefix}_lidar_imu" type="imu">
+        <always_on>true</always_on>
+        <update_rate>100</update_rate>
+        <!-- Mid-360内蔵IMUとして扱えるよう、IMU topicとframeをLiDAR個体に紐付ける。 -->
+        <plugin filename="libgazebo_ros_imu_sensor.so" name="${prefix}_gazebo_ros_imu_sensor">
+          <ros>
+            <namespace>/</namespace>
+            <remapping>~/out:=${imu_topic}</remapping>
+          </ros>
+          <frame_name>${prefix}_lidar_imu_link</frame_name>
+        </plugin>
+      </sensor>
+    </gazebo>
+  </xacro:macro>
+  <xacro:macro name="mid360_lidar" params="prefix x y z roll pitch yaw enable_imu:=false imu_topic:=/imu/data">
     <link name="${prefix}_lidar_link">
       <visual>
@@ -85,4 +105,16 @@
       <xacro:box_inertia mass="0.265" x="${mid360_depth}" y="${mid360_width}" z="${mid360_height}" />
     </link>
+    <link name="${prefix}_lidar_imu_link">
+      <visual>
+        <origin xyz="0 0 0" rpy="0 0 0" />
+        <geometry>
+          <box size="${mid360_imu_size} ${mid360_imu_size} ${mid360_imu_size}" />
+        </geometry>
+        <material name="imu_green">
+          <color rgba="0.0 0.35 0.18 1.0" />
+        </material>
+      </visual>
+      <xacro:box_inertia mass="0.01" x="${mid360_imu_size}" y="${mid360_imu_size}" z="${mid360_imu_size}" />
+    </link>
     <joint name="${prefix}_lidar_joint" type="fixed">
       <parent link="base_link" />
@@ -90,6 +122,15 @@
       <origin xyz="${x} ${y} ${z}" rpy="${roll} ${pitch} ${yaw}" />
     </joint>
+    <joint name="${prefix}_lidar_imu_joint" type="fixed">
+      <parent link="${prefix}_lidar_link" />
+      <child link="${prefix}_lidar_imu_link" />
+      <!-- 公式Mid-360 manual p.15のIMU chip位置をpoint cloud coordinates基準で反映する。 -->
+      <origin xyz="${mid360_imu_x} ${mid360_imu_y} ${mid360_imu_z}" rpy="0 0 0" />
+    </joint>
     <xacro:if value="$(arg use_sim)">
       <xacro:mid360_gazebo_sensor prefix="${prefix}" />
+      <xacro:if value="${enable_imu}">
+        <xacro:mid360_gazebo_imu prefix="${prefix}" imu_topic="${imu_topic}" />
+      </xacro:if>
     </xacro:if>
   </xacro:macro>

File: ros2_ws/src/ai_ship_robot_description/urdf/lidar/patterns/lidar_pattern_dual_out38.urdf.xacro (robot description, xacro)
@@ -19,5 +19,7 @@
     roll="${lidar_roll}"
     pitch="${lidar_pitch}"
-    yaw="${lidar_outward_yaw}" />
+    yaw="${lidar_outward_yaw}"
+    enable_imu="true"
+    imu_topic="/left_lidar/imu" />
   <xacro:mid360_lidar
     prefix="right"

File: ros2_ws/src/ai_ship_robot_description/urdf/lidar/patterns/lidar_pattern_dual_updown.urdf.xacro (robot description, xacro)
@@ -20,5 +20,7 @@
     roll="${lidar_roll}"
     pitch="${left_lidar_pitch}"
-    yaw="${lidar_yaw}" />
+    yaw="${lidar_yaw}"
+    enable_imu="true"
+    imu_topic="/left_lidar/imu" />
   <xacro:mid360_lidar
     prefix="right"
