Commit message: とりこみ

File: sim/ros2_ws/src/ai_ship_robot_description/urdf/ai_ship_robot.urdf.xacro (robot description, xacro)
@@ -8,9 +8,8 @@
   <xacro:property name="base_height" value="0.37" />
   <xacro:property name="ground_clearance" value="0.03" />
-  <xacro:property name="wheel_radius" value="0.10" />
-  <xacro:property name="wheel_width" value="0.08" />
-  <xacro:property name="wheel_separation" value="${base_width - wheel_width}" />
-  <xacro:property name="wheel_x_offset" value="${base_length / 2.0 - wheel_radius - 0.02}" />
-  <xacro:property name="base_center_z" value="${ground_clearance - wheel_radius + base_height / 2.0}" />
+  <xacro:property name="omni_wheel_radius" value="0.10" />
+  <xacro:property name="omni_wheel_separation" value="${base_width - omni_wheel_radius * 2.0 * 0.4}" />
+  <xacro:property name="omni_wheel_x_offset" value="${base_length / 2.0 - omni_wheel_radius - 0.02}" />
+  <xacro:property name="base_center_z" value="${ground_clearance - omni_wheel_radius + base_height / 2.0}" />
   <xacro:property name="arm_robot_body_length" value="0.62" />
   <xacro:property name="arm_robot_body_width" value="0.62" />
@@ -59,10 +58,10 @@
     </inertial>
   </xacro:macro>
-  <xacro:macro name="drive_wheel" params="prefix x_position y_position">
-    <link name="${prefix}_wheel_link">
-      <visual>
-        <origin xyz="0 0 0" rpy="${pi / 2.0} 0 0" />
-        <geometry>
-          <cylinder radius="${wheel_radius}" length="${wheel_width}" />
+  <xacro:macro name="support_omni_wheel" params="prefix x_position y_position">
+    <link name="${prefix}_omni_wheel_link">
+      <visual>
+        <origin xyz="0 0 0" rpy="0 0 0" />
+        <geometry>
+          <sphere radius="${omni_wheel_radius}" />
         </geometry>
         <material name="dark_gray">
@@ -71,18 +70,22 @@
       </visual>
       <collision>
-        <origin xyz="0 0 0" rpy="${pi / 2.0} 0 0" />
-        <geometry>
-          <cylinder radius="${wheel_radius}" length="${wheel_width}" />
-        </geometry>
-      </collision>
-      <xacro:cylinder_inertia mass="1.2" radius="${wheel_radius}" length="${wheel_width}" axis="y" />
-    </link>
-    <joint name="${prefix}_wheel_joint" type="continuous">
+        <origin xyz="0 0 0" rpy="0 0 0" />
+        <geometry>
+          <sphere radius="${omni_wheel_radius}" />
+        </geometry>
+      </collision>
+      <xacro:box_inertia
+        mass="1.2"
+        x="${omni_wheel_radius * 2.0}"
+        y="${omni_wheel_radius * 2.0}"
+        z="${omni_wheel_radius * 2.0}" />
+    </link>
+    <joint name="${prefix}_omni_wheel_joint" type="fixed">
       <parent link="base_link" />
-      <child link="${prefix}_wheel_link" />
+      <child link="${prefix}_omni_wheel_link" />
       <origin xyz="${x_position} ${y_position} 0" rpy="0 0 0" />
-      <axis xyz="0 1 0" />
-    </joint>
-    <gazebo reference="${prefix}_wheel_link">
+    </joint>
+    <!-- 支持球として扱うため、見た目と接地判定だけを残して駆動自由度は持たせない。 -->
+    <gazebo reference="${prefix}_omni_wheel_link">
       <material>Gazebo/Black</material>
       <mu1>1.0</mu1>
@@ -191,5 +194,5 @@
     <parent link="base_footprint" />
     <child link="base_link" />
-    <origin xyz="0 0 ${wheel_radius}" rpy="0 0 0" />
+    <origin xyz="0 0 ${omni_wheel_radius}" rpy="0 0 0" />
   </joint>
   <link name="base_link">
@@ -211,8 +214,9 @@
     <xacro:box_inertia mass="28.0" x="${base_length}" y="${base_width}" z="${base_height}" />
   </link>
-  <xacro:drive_wheel prefix="left_front" x_position="${wheel_x_offset}" y_position="${wheel_separation / 2.0}" />
-  <xacro:drive_wheel prefix="left_rear" x_position="${-wheel_x_offset}" y_position="${wheel_separation / 2.0}" />
-  <xacro:drive_wheel prefix="right_front" x_position="${wheel_x_offset}" y_position="${-wheel_separation / 2.0}" />
-  <xacro:drive_wheel prefix="right_rear" x_position="${-wheel_x_offset}" y_position="${-wheel_separation / 2.0}" />
+  <!-- 旧車輪位置に支持球を置き、本体高さを維持したままオムニホイール相当の外形に置き換える。 -->
+  <xacro:support_omni_wheel prefix="left_front" x_position="${omni_wheel_x_offset}" y_position="${omni_wheel_separation / 2.0}" />
+  <xacro:support_omni_wheel prefix="left_rear" x_position="${-omni_wheel_x_offset}" y_position="${omni_wheel_separation / 2.0}" />
+  <xacro:support_omni_wheel prefix="right_front" x_position="${omni_wheel_x_offset}" y_position="${-omni_wheel_separation / 2.0}" />
+  <xacro:support_omni_wheel prefix="right_rear" x_position="${-omni_wheel_x_offset}" y_position="${-omni_wheel_separation / 2.0}" />
   <xacro:fixed_arm_robot_fixture />
   <!-- 起動時に指定された配置ファイルを読み込み、URDF編集なしでLiDARパターンを切り替える。 -->
@@ -263,6 +267,7 @@
       <sensor name="imu" type="imu">
         <always_on>true</always_on>
-        <update_rate>100</update_rate>
+        <update_rate>200</update_rate>
         <plugin filename="libgazebo_ros_imu_sensor.so" name="gazebo_ros_imu_sensor">
+          <updateRateHZ>200.0</updateRateHZ>
           <ros>
             <namespace>/</namespace>

File: sim/ros2_ws/src/ai_ship_robot_description/urdf/lidar/models/mid360_lidar.urdf.xacro (robot description, xacro)
@@ -19,5 +19,5 @@
         <always_on>true</always_on>
         <visualize>false</visualize>
-        <update_rate>10</update_rate>
+        <update_rate>5</update_rate>
         <!-- Livox pluginの要求に合わせ、可視化用のray設定とCSV走査設定を同居させる。 -->
         <plugin name="${prefix}_livox_plugin" filename="libros2_livox.so">
@@ -74,7 +74,8 @@
       <sensor name="${prefix}_lidar_imu" type="imu">
         <always_on>true</always_on>
-        <update_rate>100</update_rate>
+        <update_rate>200</update_rate>
         <!-- Mid-360内蔵IMUとして扱えるよう、IMU topicとframeをLiDAR個体に紐付ける。 -->
         <plugin filename="libgazebo_ros_imu_sensor.so" name="${prefix}_gazebo_ros_imu_sensor">
+          <updateRateHZ>200.0</updateRateHZ>
           <ros>
             <namespace>/</namespace>

File: sim/ros2_ws/src/ai_ship_robot_description/urdf/lidar/patterns/lidar_pattern_dual_out38.urdf.xacro (robot description, xacro)
@@ -8,5 +8,5 @@
   <xacro:property name="lidar_right_y" value="${-lidar_left_y}" />
   <xacro:property name="lidar_ground_height" value="0.150" />
-  <xacro:property name="lidar_z" value="${lidar_ground_height - wheel_radius}" />
+  <xacro:property name="lidar_z" value="${lidar_ground_height}" />
   <xacro:property name="lidar_roll" value="0.0" />
   <xacro:property name="lidar_pitch" value="${90.0 * deg_to_rad}" />
@@ -29,4 +29,6 @@
     roll="${lidar_roll}"
     pitch="${lidar_pitch}"
-    yaw="${-lidar_outward_yaw}" />
+    yaw="${-lidar_outward_yaw}"
+    enable_imu="true"
+    imu_topic="/right_lidar/imu" />
 </robot>

File: sim/ros2_ws/src/ai_ship_robot_description/urdf/lidar/patterns/lidar_pattern_dual_updown.urdf.xacro (robot description, xacro)
@@ -8,5 +8,5 @@
   <xacro:property name="lidar_right_y" value="${-lidar_left_y}" />
   <xacro:property name="lidar_ground_height" value="0.150" />
-  <xacro:property name="lidar_z" value="${lidar_ground_height - wheel_radius}" />
+  <xacro:property name="lidar_z" value="${lidar_ground_height}" />
   <xacro:property name="lidar_roll" value="0.0" />
   <xacro:property name="lidar_yaw" value="0.0" />
@@ -30,4 +30,6 @@
     roll="${lidar_roll}"
     pitch="${right_lidar_pitch}"
-    yaw="${lidar_yaw}" />
+    yaw="${lidar_yaw}"
+    enable_imu="true"
+    imu_topic="/right_lidar/imu" />
 </robot>

Commit message: Livox CustomMsg基準のSLAM導線を整理
- 複数LiDAR fusionをCustomMsg出力に統一
- LIO-SAMにhybrid登録点群、cloudQueue排出待ち、publish制御を追加
- PCD map saverをodometry/path同期のsubmap保存方式へ更新
- Gazebo simulationとrosbag導線を複数LiDAR topic構成へ追従
- 走行シナリオ、環境セットアップ、本番配布スクリプトを整備

File: sim/ros2_ws/src/ai_ship_robot_description/urdf/ai_ship_robot.urdf.xacro (robot description, xacro)
@@ -2,5 +2,5 @@
 <robot xmlns:xacro="http://www.ros.org/wiki/xacro" name="ai_ship_robot">
   <xacro:arg name="use_sim" default="true" />
-  <xacro:arg name="lidar_pattern_file" default="lidar_pattern_dual_updown.urdf.xacro" />
+  <xacro:arg name="lidar_pattern_file" default="lidar_pattern_dual_front_updown.urdf.xacro" />
   <xacro:arg name="publish_odom_tf" default="true" />
   <xacro:property name="base_length" value="0.72" />

File: sim/ros2_ws/src/ai_ship_robot_description/urdf/lidar/models/mid360_lidar.urdf.xacro (robot description, xacro)
@@ -15,6 +15,6 @@
   <xacro:property name="mid360_imu_size" value="0.015" />
   <xacro:macro name="mid360_gazebo_sensor" params="prefix">
-    <gazebo reference="${prefix}_lidar_link">
-      <sensor name="${prefix}_lidar_link" type="ray">
+    <gazebo reference="${prefix}_link">
+      <sensor name="${prefix}_link" type="ray">
         <always_on>true</always_on>
         <visualize>false</visualize>
@@ -64,6 +64,7 @@
           <csv_file_name>$(find ros2_livox_simulation)/scan_mode/mid360.csv</csv_file_name>
           <topic>${prefix}_livox</topic>
-          <custom_topic>/${prefix}_lidar/custom</custom_topic>
-          <pointcloud2_topic>/${prefix}_lidar/points</pointcloud2_topic>
+          <custom_topic>/${prefix}/custom</custom_topic>
+          <pointcloud2_topic>/${prefix}/points</pointcloud2_topic>
+          <enable_pointcloud2>false</enable_pointcloud2>
         </plugin>
       </sensor>
@@ -71,6 +72,6 @@
   </xacro:macro>
   <xacro:macro name="mid360_gazebo_imu" params="prefix imu_topic">
-    <gazebo reference="${prefix}_lidar_imu_link">
-      <sensor name="${prefix}_lidar_imu" type="imu">
+    <gazebo reference="${prefix}_imu_link">
+      <sensor name="${prefix}_imu" type="imu">
         <always_on>true</always_on>
         <update_rate>200</update_rate>
@@ -82,5 +83,5 @@
             <remapping>~/out:=${imu_topic}</remapping>
           </ros>
-          <frame_name>${prefix}_lidar_imu_link</frame_name>
+          <frame_name>${prefix}_imu_link</frame_name>
         </plugin>
       </sensor>
@@ -88,5 +89,5 @@
   </xacro:macro>
   <xacro:macro name="mid360_lidar" params="prefix x y z roll pitch yaw enable_imu:=false imu_topic:=/imu/data">
-    <link name="${prefix}_lidar_link">
+    <link name="${prefix}_link">
       <visual>
         <origin xyz="0 0 0" rpy="0 0 0" />
@@ -106,5 +107,5 @@
       <xacro:box_inertia mass="0.265" x="${mid360_depth}" y="${mid360_width}" z="${mid360_height}" />
     </link>
-    <link name="${prefix}_lidar_imu_link">
+    <link name="${prefix}_imu_link">
       <visual>
         <origin xyz="0 0 0" rpy="0 0 0" />
@@ -118,12 +119,12 @@
       <xacro:box_inertia mass="0.01" x="${mid360_imu_size}" y="${mid360_imu_size}" z="${mid360_imu_size}" />
     </link>
-    <joint name="${prefix}_lidar_joint" type="fixed">
+    <joint name="${prefix}_joint" type="fixed">
       <parent link="base_link" />
-      <child link="${prefix}_lidar_link" />
+      <child link="${prefix}_link" />
       <origin xyz="${x} ${y} ${z}" rpy="${roll} ${pitch} ${yaw}" />
     </joint>
-    <joint name="${prefix}_lidar_imu_joint" type="fixed">
-      <parent link="${prefix}_lidar_link" />
-      <child link="${prefix}_lidar_imu_link" />
+    <joint name="${prefix}_imu_joint" type="fixed">
+      <parent link="${prefix}_link" />
+      <child link="${prefix}_imu_link" />
       <!-- 公式Mid-360 manual p.15のIMU chip位置をpoint cloud coordinates基準で反映する。 -->
       <origin xyz="${mid360_imu_x} ${mid360_imu_y} ${mid360_imu_z}" rpy="0 0 0" />

File: sim/ros2_ws/src/ai_ship_robot_description/urdf/lidar/patterns/lidar_pattern_dual_out38.urdf.xacro (robot description, xacro)
@@ -13,5 +13,5 @@
   <xacro:property name="lidar_outward_yaw" value="${38.0 * deg_to_rad}" />
   <xacro:mid360_lidar
-    prefix="left"
+    prefix="lidar1"
     x="${lidar_front_x}"
     y="${lidar_left_y}"
@@ -21,7 +21,7 @@
     yaw="${lidar_outward_yaw}"
     enable_imu="true"
-    imu_topic="/left_lidar/imu" />
+    imu_topic="/lidar1/imu" />
   <xacro:mid360_lidar
-    prefix="right"
+    prefix="lidar2"
     x="${lidar_front_x}"
     y="${lidar_right_y}"
@@ -31,4 +31,4 @@
     yaw="${-lidar_outward_yaw}"
     enable_imu="true"
-    imu_topic="/right_lidar/imu" />
+    imu_topic="/lidar2/imu" />
 </robot>

File: sim/ros2_ws/src/ai_ship_robot_description/urdf/lidar/patterns/lidar_pattern_dual_updown.urdf.xacro (robot description, xacro)
@@ -11,25 +11,25 @@
   <xacro:property name="lidar_roll" value="0.0" />
   <xacro:property name="lidar_yaw" value="0.0" />
-  <xacro:property name="left_lidar_pitch" value="${120.0 * deg_to_rad}" />
-  <xacro:property name="right_lidar_pitch" value="${30.0 * deg_to_rad}" />
+  <xacro:property name="lidar1_pitch" value="${120.0 * deg_to_rad}" />
+  <xacro:property name="lidar2_pitch" value="${30.0 * deg_to_rad}" />
   <xacro:mid360_lidar
-    prefix="left"
+    prefix="lidar1"
     x="${lidar_front_x}"
     y="${lidar_left_y}"
     z="${lidar_z}"
     roll="${lidar_roll}"
-    pitch="${left_lidar_pitch}"
+    pitch="${lidar1_pitch}"
     yaw="${lidar_yaw}"
     enable_imu="true"
-    imu_topic="/left_lidar/imu" />
+    imu_topic="/lidar1/imu" />
   <xacro:mid360_lidar
-    prefix="right"
+    prefix="lidar2"
     x="${lidar_front_x}"
     y="${lidar_right_y}"
     z="${lidar_z}"
     roll="${lidar_roll}"
-    pitch="${right_lidar_pitch}"
+    pitch="${lidar2_pitch}"
     yaw="${lidar_yaw}"
     enable_imu="true"
-    imu_topic="/right_lidar/imu" />
+    imu_topic="/lidar2/imu" />
 </robot>

Commit message: 20260623_2037 取り込み

File: sim/ros2_ws/src/ai_ship_robot_description/urdf/ai_ship_robot.urdf.xacro (robot description, xacro)
@@ -2,12 +2,12 @@
 <robot xmlns:xacro="http://www.ros.org/wiki/xacro" name="ai_ship_robot">
   <xacro:arg name="use_sim" default="true" />
-  <xacro:arg name="lidar_pattern_file" default="lidar_pattern_dual_front_updown.urdf.xacro" />
+  <xacro:arg name="lidar_pattern_file" default="lidar_pattern_dual_opposit.urdf.xacro" />
   <xacro:arg name="publish_odom_tf" default="true" />
   <xacro:property name="base_length" value="0.72" />
   <xacro:property name="base_width" value="0.72" />
-  <xacro:property name="base_height" value="0.37" />
+  <xacro:property name="base_height" value="0.30" />
   <xacro:property name="ground_clearance" value="0.03" />
-  <xacro:property name="omni_wheel_radius" value="0.10" />
-  <xacro:property name="omni_wheel_separation" value="${base_width - omni_wheel_radius * 2.0 * 0.4}" />
+  <xacro:property name="omni_wheel_radius" value="0.05" />
+  <xacro:property name="omni_wheel_separation" value="${base_width - omni_wheel_radius * 2.0 -0.15}" />
   <xacro:property name="omni_wheel_x_offset" value="${base_length / 2.0 - omni_wheel_radius - 0.02}" />
   <xacro:property name="base_center_z" value="${ground_clearance - omni_wheel_radius + base_height / 2.0}" />
@@ -200,7 +200,9 @@
   <link name="base_link">
     <visual>
-      <origin xyz="0 0 ${base_center_z}" rpy="0 0 0" />
-      <geometry>
-        <box size="${base_length} ${base_width} ${base_height}" />
+      <!-- 本体の物理近似は箱のまま維持しつつ、表示だけ実機外形メッシュへ置き換える。 -->
+      <origin xyz="0 0 ${base_center_z - base_height / 2.0}" rpy="0 0 0" />
+      <geometry>
+        <mesh filename="package://ai_ship_robot_description/mesh/AiTran500_L24970.stl"
+              scale="0.001 0.001 0.001"/>
       </geometry>
       <material name="navy_blue">

File: sim/ros2_ws/src/ai_ship_robot_description/urdf/lidar/models/mid360_lidar.urdf.xacro (robot description, xacro)
@@ -3,7 +3,7 @@
   <xacro:arg name="half_lidar_resolution" default="false" />
   <xacro:arg name="quarter_lidar_resolution" default="false" />
-  <xacro:property name="mid360_depth" value="0.060" />
+  <xacro:property name="mid360_depth" value="0.065" />
   <xacro:property name="mid360_width" value="0.065" />
-  <xacro:property name="mid360_height" value="0.065" />
+  <xacro:property name="mid360_height" value="0.060" />
   <xacro:property name="mid360_samples" value="40000" />
   <xacro:property name="mid360_downsample" value="1" />
@@ -91,7 +91,9 @@
     <link name="${prefix}_link">
       <visual>
-        <origin xyz="0 0 0" rpy="0 0 0" />
+        <!-- LiDAR配置用joint姿勢を変えずに済むよう、見た目の差し替えはvisual側だけで閉じ込める。 -->
+        <origin xyz="0 ${-mid360_width / 2.0} ${-mid360_height / 2.0}" rpy="${pi / 2.0} 0 ${pi / 2.0}" />
         <geometry>
-          <box size="${mid360_depth} ${mid360_width} ${mid360_height}" />
+          <mesh filename="package://ai_ship_robot_description/mesh/mid360.stl"
+                scale="0.001 0.001 0.001" />
         </geometry>
         <material name="sensor_black">
