Commit message: とりこみ

File: sim/ros2_ws/src/ai_ship_robot_description/urdf/lidar/models/mid360_lidar.urdf.xacro (robot description, xacro)
@@ -91,6 +91,6 @@
     <link name="${prefix}_link">
       <visual>
-        <!-- 従来の箱形状を簡略meshとして参照し、LiDAR frame上の見え方を維持する。 -->
-        <origin xyz="0 0 0" rpy="0 0 0" />
+        <!-- LiDAR配置用joint姿勢を変えずに済むよう、見た目の差し替えはvisual側だけで閉じ込める。 -->
+        <origin xyz="0 ${-mid360_width / 2.0} ${-mid360_height / 2.0}" rpy="${pi / 2.0} 0 ${pi / 2.0}" />
         <geometry>
           <mesh filename="package://ai_ship_robot_description/mesh/mid360.stl"
